Commit message: ik added

File: ros2_ws/src/my_package/urdf/arm.urdf.xacro (robot description, xacro)
@@ -132,4 +132,10 @@
     <limit lower="0.0" upper="0.03" velocity="0.1" effort="5.0"/>
   </joint>
+  <link name="tool_tip"/>
+  <joint name="tool_tip_joint" type="fixed">
+    <parent link="gripper_base_link"/>
+    <child link="tool_tip"/>
+    <origin xyz="0 0 0.06"/>
+  </joint>
   <!-- ros2_control -->
   <ros2_control name="ArmSystem" type="system">
